File: PCB/cougar mmjoy.brd (EAGLE design)
At the start: 50.5 x 38.1 mm, 6 parts, among them J1 X AXIS, J2 Y AXIS, J3 STICK BTNS, J4 USB-B, J5 ARDUINO, U1 ARDUINO_PRO_MICRO

Commit message: Updated SketchUp models
Created detailed SketchUp models, concept graphic
Parts:
- moved J1 24.3 mm to (25.4, 29.2), turned to 0 degrees
- moved J3 11.7 mm to (26.7, 15.2), turned to 0 degrees
- moved J2 2.84 mm to (25.4, 21.6), turned to 0 degrees
Routing:
- net GND: track 110.7 -> 77.8 mm
- net CS_STICK: track 29.6 -> 45.0 mm
- net CS_Y_AXIS: track 22.7 -> 34.8 mm
- net MISO: track 34.7 -> 24.2 mm
- net SCK: track 32.2 -> 25.6 mm
- net VCC: track 82.5 -> 77.7 mm
- net N$4: track 22.1 -> 23.2 mm
- net N$3: track 21.9 -> 22.9 mm
- net CLK: track 31.9 -> 31.0 mm
- added copper zone on layer 1, net GND
- added copper zone on layer 16, net GND
- removed copper zone on layer 1, net N$1
- removed copper zone on layer 16, net N$2
Other:
- board text added: "CC BY NC SA"
- board text added: "github.com/mejtoogood/Cougar-MMjoy"
